Commit message: Rebase from 'upstream'

File: robots/mpo_700/mpo_700.urdf (robot description, URDF)
Before this commit: robot mpo_700, 12 links, 11 joints
Links:
- added link camera_link, mass 1e-5; collision box size=0.05 0.05 0.05; visual mesh filename=package://neo_simulation2/components/sensors/d435.dae
- added link camera_link_gazebo
- added link camera_link_optical
Joints:
- added joint camera_gazebo_joint: type fixed, parent camera_link, child camera_link_gazebo, origin xyz=0 0.015 0 rpy=0 0 0
- added joint camera_joint: type fixed, parent base_link, child camera_link, origin xyz=-0.228 0.015 0.461 rpy=0 0 3.14159, axis 0 1 0
- added joint camera_optical_joint: type fixed, parent camera_link, child camera_link_optical, origin xyz=0 0.015 0 rpy=-1.5707963267948966 0 -1.5707963267948966
